File: control_board.kicad_pcb (KiCad board)
At the start: 2 copper layers, 44.5 x 46.8 mm, 21 parts, among them IC1 ATMEGA328P-A, J1 USB_C_Receptacle, J2 AVR-ISP-6, P1 CONN_8, U1 MCP7940N-xSN, Y1 Crystal_GND23

Commit message: Update for board rev 2
Move USB connector to board edge
Move resisters to not interfere with programming header
Widen board to fit enclosure
Move programming header and USB connector away from top/bottom of board for more clearance with enclosure
Move red encoder LED to a PWM capable pin
Parts:
- moved J1 5.11 mm to (135.9, 64.5)
- moved G*** 2.54 mm to (165.6, 59.6) (x2)
- moved G*** 2.54 mm to (165.6, 59.5)
- moved R5 1.92 mm to (149.4, 33.9)
- moved R1 1.43 mm to (150.2, 31.2)
- moved J2 1.27 mm to (143.8, 32.5)
Connections:
- IC1 pad 14: Net-(IC1-Pad14) -> /Red
- IC1 pad 2: /Red -> Net-(IC1-Pad2)
Routing:
- net /Red: track 29.3 -> 11.8 mm
- net +5V: track 62.1 -> 51.0 mm, vias 5 -> 4
- net GND: track 66.9 -> 56.6 mm
- net /Reset: track 26.7 -> 29.6 mm
- net Net-(J2-Pad1): track 4.05 -> 6.02 mm
- net Net-(J2-Pad3): track 9.42 -> 8.65 mm
- net Net-(IC1-Pad16): track 25.9 -> 26.5 mm
- net Net-(J2-Pad4): track 8.95 -> 8.37 mm
Other:
- board size 44.5 x 46.8 mm -> 47 x 46.8 mm
